File: BLDC.sch (EAGLE design)
At the start: 56 parts, among them IC1 A4960, Q1 AUIR1324S, Q2 AUIR1324S, Q3 AUIR1324S, Q4 AUIR1324S, Q5 AUIR1324S, Q6 AUIR1324S, U1 MC34063, U2 LM1117-5.0

Commit message: change some values, move R5 to reduce risk of shorting it
Parts:
- C1, C2, C3: value 1uF -> 10uF
- C21, C22, C5: value 1uF -> 100nF
- C4: value 1uF -> 220nF
Changed lines of the file:
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@@
 <part name="P+1" library="supply1" deviceset="+12V" device=""/>
 <part name="GND1" library="supply1" deviceset="GND" device=""/>
-<part name="C1" library="rcl" deviceset="C-EU" device="C0603K" value="1uF"/>
-<part name="C2" library="rcl" deviceset="C-EU" device="C0603K" value="1uF"/>
-<part name="C3" library="rcl" deviceset="C-EU" device="C0603K" value="1uF"/>
-<part name="C4" library="rcl" deviceset="C-EU" device="C0603K" value="1uF"/>
-<part name="C5" library="rcl" deviceset="C-EU" device="C0603K" value="1uF"/>
+<part name="C1" library="rcl" deviceset="C-EU" device="C0603K" value="10uF"/>
+<part name="C2" library="rcl" deviceset="C-EU" device="C0603K" value="10uF"/>
+<part name="C3" library="rcl" deviceset="C-EU" device="C0603K" value="10uF"/>
+<part name="C4" library="rcl" deviceset="C-EU" device="C0603K" value="220nF"/>
+<part name="C5" library="rcl" deviceset="C-EU" device="C0603K" value="100nF"/>
 <part name="GND2" library="supply1" deviceset="GND" device=""/>
 <part name="P+2" library="supply1" deviceset="+12V" device=""/>
@@
 <part name="R6" library="rcl" deviceset="R-EU_" device="R0603" value="22R"/>
 <part name="R7" library="rcl" deviceset="R-EU_" device="R0603" value="22R"/>
-<part name="C21" library="rcl" deviceset="C-EU" device="C0603K" value="1uF"/>
+<part name="C21" library="rcl" deviceset="C-EU" device="C0603K" value="100nF"/>
 <part name="GND4" library="supply1" deviceset="GND" device=""/>
 <part name="JP1" library="pinhead" deviceset="PINHD-2X10" device=""/>
-<part name="C22" library="rcl" deviceset="C-EU" device="C0603K" value="1uF"/>
+<part name="C22" library="rcl" deviceset="C-EU" device="C0603K" value="100nF"/>
 <part name="GND5" library="supply1" deviceset="GND" device=""/>
 <part name="L2" library="microbuilder" deviceset="INDUCTOR" device="0603" value="bead"/>
